File: circuits/fan-control-nano/fan-control-nano.kicad_sch (KiCad schematic)
At the start: 21 parts, among them J1 Conn_01x02_Pin, J2 Conn_01x03_Pin, J3 Screw_Terminal_12V, M1 Fan_4pin, M2 Fan_4pin, M3 Fan, M4 Fan, M5 Fan, Q1 BD139, Q2 BD139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

Commit message: Update nano circuit, add rpi circuit, update readme.
Parts:
- added U3: AD22100KTZ, Package_SO:SOIC-8_3.9x4.9mm_P1.27mm, symbol AD22100:AD22100KTZ
Connections:
- net GND2: now also U3.4 (GND)
- net at A1.27 (+5V), R4.1, TH1.1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: now also U3.8 (+V_{S})
- net at A1.19 (A0): now also U3.1 (V_{OUT})
Other:
- moved on the sheet: U2
